Commit message: Imported upstream version '3.0.0' of 'upstream'

File: create_description/urdf/create_1.urdf.xacro (robot description, xacro)
@@ -1,8 +1,7 @@
 <?xml version="1.0" ?>
-<robot name="create_1"
-  xmlns:xacro="http://ros.org/wiki/xacro">
+<robot name="create_1" xmlns:xacro="http://ros.org/wiki/xacro">
   <xacro:include filename="$(find create_description)/urdf/create_base.urdf.xacro" />
   <xacro:include filename="$(find create_description)/urdf/create_1_gazebo.urdf.xacro" />
-  <xacro:create_base wheel_separation="0.26" base_diameter="0.3302" version="1">
+  <xacro:create_base wheel_separation="0.26" base_diameter="0.3302">
     <mesh filename="package://create_description/meshes/create_1.dae" />
   </xacro:create_base>

File: create_description/urdf/create_2.urdf.xacro (robot description, xacro)
@@ -1,8 +1,7 @@
 <?xml version="1.0" ?>
-<robot name="create_2"
-  xmlns:xacro="http://ros.org/wiki/xacro">
+<robot name="create_2" xmlns:xacro="http://ros.org/wiki/xacro">
   <xacro:include filename="$(find create_description)/urdf/create_base.urdf.xacro" />
   <xacro:include filename="$(find create_description)/urdf/create_2_gazebo.urdf.xacro" />
-  <xacro:create_base wheel_separation="0.235" base_diameter="0.3485" version="2">
+  <xacro:create_base wheel_separation="0.235" base_diameter="0.3485">
     <mesh filename="package://create_description/meshes/create_2.dae" />
   </xacro:create_base>

File: create_description/urdf/create_base.urdf.xacro (robot description, xacro)
@@ -4,23 +4,23 @@
   <xacro:macro name="create_wheel" params="prefix y_offset wheel_radius wheel_width">
     <link name="${prefix}_wheel_link">
-      <inertial>
-        <origin xyz="0 0 0" />
-        <mass value="0.01" />
-        <inertia ixx="0.001" ixy="0.0" ixz="0.0" iyy="0.001" iyz="0.0" izz="0.001" />
-      </inertial>
-      <visual>
-        <origin xyz="0 0 0" rpy="0 ${PI/2} ${PI/2}" />
-        <geometry>
-          <cylinder radius="${wheel_radius}" length="${wheel_width}" />
-        </geometry>
-      </visual>
-      <collision>
-        <origin xyz="0 0 0" rpy="0 ${PI/2} ${PI/2}" />
-        <geometry>
-          <cylinder radius="${wheel_radius}" length="${wheel_width}" />
-        </geometry>
-      </collision>
-    </link>
-    <joint name="${prefix}_wheel_joint" type="continuous">
+    <inertial>
+      <origin xyz="0 0 0" />
+      <mass value="0.01" />
+      <inertia ixx="0.001" ixy="0.0" ixz="0.0" iyy="0.001" iyz="0.0" izz="0.001" />
+    </inertial>
+    <visual>
+      <origin xyz="0 0 0" rpy="0 ${PI/2} ${PI/2}" />
+      <geometry>
+        <cylinder radius="${wheel_radius}" length="${wheel_width}" />
+      </geometry>
+    </visual>
+    <collision>
+      <origin xyz="0 0 0" rpy="0 ${PI/2} ${PI/2}" />
+      <geometry>
+        <cylinder radius="${wheel_radius}" length="${wheel_width}" />
+      </geometry>
+    </collision>
+    </link>
+   <joint name="${prefix}_wheel_joint" type="continuous">
       <origin xyz="0 ${y_offset} 0.015" rpy="0 0 0" />
       <parent link="base_link" />
@@ -29,77 +29,74 @@
     </joint>
   </xacro:macro>
-  <xacro:macro name="create_base" params="diffdrive_update_rate:=40 wheel_separation wheel_radius:=0.036 wheel_width:=0.024 wheel_torque:=1.0 wheel_accel:=1.8 mass_kg:=3.5 base_diameter version *mesh">
+  <xacro:macro name="create_base" params="diffdrive_update_rate:=40 wheel_separation wheel_radius:=0.036 wheel_width:=0.024 wheel_torque:=1.0 wheel_accel:=1.8 mass_kg:=3.5 base_diameter *mesh">
     <xacro:include filename="$(find create_description)/urdf/create_base_gazebo.urdf.xacro" />
-    <material name="green">
-      <color rgba="0 0.8 0 1"/>
-    </material>
     <link name="base_footprint">
-      <visual>
-        <origin xyz="0 0 0" rpy="0 0 0" />
-        <geometry>
-          <box size="0.001 0.001 0.001" />
-        </geometry>
-        <material name="green" />
-      </visual>
-      <collision>
-        <origin xyz="0 0 0.017" rpy="0 0 0" />
-        <geometry>
-          <box size="0.001 0.001 0.001" />
-        </geometry>
-      </collision>
+    <visual>
+      <origin xyz="0 0 0" rpy="0 0 0" />
+      <geometry>
+        <box size="0.001 0.001 0.001" />
+      </geometry>
+      <material name="Green" />
+    </visual>
+    <collision>
+      <origin xyz="0 0 0.017" rpy="0 0 0" />
+      <geometry>
+        <box size="0.001 0.001 0.001" />
+      </geometry>
+    </collision>
     </link>
     <link name="base_link">
-      <inertial>
-        <mass value="2" />
-        <origin xyz="0 0 0.0" />
-        <inertia ixx="0.01" ixy="0.0" ixz="0.0" iyy="0.01" iyz="0.0" izz="0.5" />
-      </inertial>
-      <visual>
-        <origin xyz=" 0 0 0.0308" rpy="0 0 0" />
-        <geometry>
-          <xacro:insert_block name="mesh" />
-        </geometry>
-      </visual>
-      <collision>
-        <origin xyz="0.0 0.0 0.0308" rpy="0 0 0" />
-        <geometry>
-          <cylinder length="0.0611632" radius="0.16495" />
-        </geometry>
-      </collision>
+    <inertial>
+      <mass value="2" />
+      <origin xyz="0 0 0.0" />
+      <inertia ixx="0.01" ixy="0.0" ixz="0.0" iyy="0.01" iyz="0.0" izz="0.5" />
+    </inertial>
+    <visual>
+      <origin xyz=" 0 0 0.0308" rpy="0 0 0" />
+      <geometry>
+        <xacro:insert_block name="mesh" />
+      </geometry>
+    </visual>
+    <collision>
+      <origin xyz="0.0 0.0 0.0308" rpy="0 0 0" />
+      <geometry>
+        <cylinder length="0.0611632" radius="0.16495" />
+      </geometry>
+    </collision>
     </link>
     <link name="wall_sensor_link">
-      <inertial>
-        <mass value="0.01" />
-        <origin xyz="0 0 0" />
-        <inertia ixx="0.001" ixy="0.0" ixz="0.0" iyy="0.001" iyz="0.0" izz="0.001" />
-      </inertial>
+    <inertial>
+      <mass value="0.01" />
+      <origin xyz="0 0 0" />
+      <inertia ixx="0.001" ixy="0.0" ixz="0.0" iyy="0.001" iyz="0.0" izz="0.001" />
+    </inertial>
     </link>
     <link name="left_cliff_sensor_link">
-      <inertial>
-        <mass value="0.01" />
-        <origin xyz="0 0 0" />
-        <inertia ixx="0.001" ixy="0.0" ixz="0.0" iyy="0.001" iyz="0.0" izz="0.001" />
-      </inertial>
+    <inertial>
+      <mass value="0.01" />
+      <origin xyz="0 0 0" />
+      <inertia ixx="0.001" ixy="0.0" ixz="0.0" iyy="0.001" iyz="0.0" izz="0.001" />
+    </inertial>
     </link>
     <link name="right_cliff_sensor_link">
-      <inertial>
-        <mass value="0.01" />
-        <origin xyz="0 0 0" />
-        <inertia ixx="0.001" ixy="0.0" ixz="0.0" iyy="0.001" iyz="0.0" izz="0.001" />
-      </inertial>
+    <inertial>
+      <mass value="0.01" />
+      <origin xyz="0 0 0" />
+      <inertia ixx="0.001" ixy="0.0" ixz="0.0" iyy="0.001" iyz="0.0" izz="0.001" />
+    </inertial>
     </link>
     <link name="leftfront_cliff_sensor_link">
-      <inertial>
-        <mass value="0.01" />
-        <origin xyz="0 0 0" />
-        <inertia ixx="1.0" ixy="0.0" ixz="0.0" iyy="0.01" iyz="0.0" izz="0.01" />
-      </inertial>
+    <inertial>
+      <mass value="0.01" />
+      <origin xyz="0 0 0" />
+      <inertia ixx="1.0" ixy="0.0" ixz="0.0" iyy="0.01" iyz="0.0" izz="0.01" />
+    </inertial>
     </link>
     <link name="rightfront_cliff_sensor_link">
-      <inertial>
-        <mass value="0.01" />
-        <origin xyz="0 0 0" />
-        <inertia ixx="0.001" ixy="0.0" ixz="0.0" iyy="0.001" iyz="0.0" izz="0.001" />
-      </inertial>
+    <inertial>
+      <mass value="0.01" />
+      <origin xyz="0 0 0" />
+      <inertia ixx="0.001" ixy="0.0" ixz="0.0" iyy="0.001" iyz="0.0" izz="0.001" />
+    </inertial>
     </link>
     <joint name="base_footprint_joint" type="fixed">
@@ -135,33 +132,10 @@
     <xacro:create_wheel prefix="left" y_offset="${wheel_separation / 2}" wheel_radius="${wheel_radius}" wheel_width="${wheel_width}"/>
     <xacro:create_wheel prefix="right" y_offset="${wheel_separation / -2}" wheel_radius="${wheel_radius}" wheel_width="${wheel_width}"/>
-    <!-- bumper sensor link -->
-    <link name="bumper_link">
-      <collision name="bumper_link_collision">
-        <origin xyz="0 0 0" rpy="0 0 0"/>
-        <geometry>
-          <mesh filename="package://create_description/meshes/bumper_${version}.dae"/>
-        </geometry>
-      </collision>
-    </link>
-    <joint name="bumper_joint" type="fixed">
-      <origin xyz="-0.0025 0 0" rpy="0 0 0" />
-      <parent link="base_link" />
-      <child link="bumper_link" />
-      <axis xyz="0 0 0" />
-    </joint>
-    <!-- omni_ir sensor link -->
-    <link name="omni_ir_link">
-    </link>
-    <joint name="omni_ir_joint" type="fixed">
-      <origin xyz="${base_diameter/2 - 0.025} 0 0.0775" rpy="0 0 0" />
-      <parent link="base_link" />
-      <child link="omni_ir_link" />
-      <axis xyz="0 0 0" />
-    </joint>
     <!--<link name="rear_wheel_link">
     <inertial>
       <origin xyz="0 0 0"/>
       <mass value="0.001" />
-      <inertia ixx="0.0001" ixy="0.0" ixz="0.0" iyy="0.0001" iyz="0.0" izz="0.0001" />
+      <inertia ixx="0.0001" ixy="0.0" ixz="0.0"
+        iyy="0.0001" iyz="0.0" izz="0.0001" />
     </inertial>
     <visual>
@@ -185,21 +159,21 @@
     </joint>-->
     <link name="front_wheel_link">
-      <inertial>
-        <origin xyz="0 0 0" />
-        <mass value="0.01" />
-        <inertia ixx="0.001" ixy="0.0" ixz="0.0" iyy="0.001" iyz="0.0" izz="0.001" />
-      </inertial>
-      <visual>
-        <origin xyz="0 0 0" rpy="0 ${PI/2} ${PI/2}" />
-        <geometry>
-          <sphere radius="0.018" />
-        </geometry>
-      </visual>
-      <collision>
-        <origin xyz="0 0 0" rpy="0 ${PI/2} ${PI/2}" />
-        <geometry>
-          <sphere radius="0.018" />
-        </geometry>
-      </collision>
+    <inertial>
+      <origin xyz="0 0 0" />
+      <mass value="0.01" />
+      <inertia ixx="0.001" ixy="0.0" ixz="0.0" iyy="0.001" iyz="0.0" izz="0.001" />
+    </inertial>
+    <visual>
+      <origin xyz="0 0 0" rpy="0 ${PI/2} ${PI/2}" />
+      <geometry>
+        <sphere radius="0.018" />
+      </geometry>
+    </visual>
+    <collision>
+      <origin xyz="0 0 0" rpy="0 ${PI/2} ${PI/2}" />
+      <geometry>
+        <sphere radius="0.018" />
+      </geometry>
+    </collision>
     </link>
     <!-- fixed because there's no transmission -->
@@ -217,9 +191,9 @@
     </joint>
     <link name="gyro_link">
-      <inertial>
-        <mass value="0.001" />
-        <origin xyz="0 0 0" rpy="0 0 0" />
-        <inertia ixx="0.0001" ixy="0" ixz="0" iyy="0.000001" iyz="0" izz="0.0001" />
-      </inertial>
+    <inertial>
+      <mass value="0.001" />
+      <origin xyz="0 0 0" rpy="0 0 0" />
+      <inertia ixx="0.0001" ixy="0" ixz="0" iyy="0.000001" iyz="0" izz="0.0001" />
+    </inertial>
     </link>
     <!-- Simulation sensors -->
@@ -228,5 +202,4 @@
     <xacro:sim_create_cliff_sensors/>
     <xacro:sim_imu/>
-    <xacro:sim_bumper/>
   </xacro:macro>
 </robot>

File: create_description/urdf/create_base_gazebo.urdf.xacro (robot description, xacro)
@@ -16,5 +16,4 @@
         <odometryFrame>odom</odometryFrame>
         <robotBaseFrame>base_footprint</robotBaseFrame>
-        <publishWheelJointState>true</publishWheelJointState>
       </plugin>
       <plugin name="p3d_base_controller" filename="libgazebo_ros_p3d.so">
@@ -75,20 +74,4 @@
         <rpyOffsets>0 0 0</rpyOffsets>
       </plugin>
-    </gazebo>
-  </xacro:macro>
-  <xacro:macro name="sim_bumper">
-    <gazebo reference="bumper_link">
-      <sensor name="sim_bumper" type="contact">
-        <alwaysOn>true</alwaysOn>
-        <updateRate>1000.0</updateRate>
-        <material>Gazebo/Red</material>
-        <contact>
-          <collision>base_footprint_fixed_joint_lump__bumper_link_collision_collision_2</collision>
-        </contact>
-        <plugin name="gazebo_ros_bumper_controller" filename="libgazebo_ros_bumper.so">
-          <bumperTopicName>bumper</bumperTopicName>
-          <frameName>bumper_link</frameName>
-        </plugin>
-      </sensor>
     </gazebo>
   </xacro:macro>
